File: PCB/optocoupler/XRTL_opto.kicad_pcb (KiCad board)
At the start: 2 copper layers, 63.5 x 86.4 mm, 30 parts, among them J10 servo1, J11 servo2, J12 infoLED, J13 USBC_5V_3A_input, J15 input, J18 divider, J2 stepper1, J3 stepper2, J4 ESP32 right, J5 ESP32 left, J6 relay2, J7 relay1, U1 TBD62003, U2 TBD62003, U3 TLP3553A, U4 TLP3553A

Commit message: changed macro control keys
Routing:
- net GND: vias 29 -> 30
Changed lines of the file:
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@@
   (via (at 96.012 65.532) (size 0.8) (drill 0.4) (layers "F.Cu" "B.Cu") (free) (net 1))
   (via (at 128.905 78.74) (size 0.8) (drill 0.4) (layers "F.Cu" "B.Cu") (free) (net 1))
+  (via (at 84.328 72.644) (size 0.8) (drill 0.4) (layers "F.Cu" "B.Cu") (free) (net 1))
   (via (at 129.54 118.872) (size 0.8) (drill 0.4) (layers "F.Cu" "B.Cu") (free) (net 1))
   (via (at 97.028 72.644) (size 0.8) (drill 0.4) (layers "F.Cu" "B.Cu") (free) (net 1))

Commit message: PCB updates
Other:
- board text added: "XRTL v1.1 Jari Domke 20/04/2023"
- board text removed: "XRTL v1.1 Jari Domke 25/01/2023"
Changed lines of the file:
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@@
       (layerselection 0x00010fc_ffffffff)
       (disableapertmacros false)
-      (usegerberextensions false)
-      (usegerberattributes true)
-      (usegerberadvancedattributes true)
-      (creategerberjobfile true)
+      (usegerberextensions true)
+      (usegerberattributes false)
+      (usegerberadvancedattributes false)
+      (creategerberjobfile false)
       (svguseinch false)
       (svgprecision 6)
@@
       (plotinvisibletext false)
       (sketchpadsonfab false)
-      (subtractmaskfromsilk false)
+      (subtractmaskfromsilk true)
       (outputformat 1)
       (mirror false)
@@
     (effects (font (size 1 1) (thickness 0.15)))
   )
-  (gr_text "XRTL v1.1\nJari Domke\n25/01/2023" (at 86.36 129.54) (layer "B.SilkS")
+  (gr_text "XRTL v1.1\nJari Domke\n20/04/2023" (at 86.36 129.54) (layer "B.SilkS")
     (effects (font (size 1 1) (thickness 0.15)) (justify left mirror))
   )
@@
     (effects (font (size 1 1) (thickness 0.15)))
   )
+  (gr_text "div" (at 124.46 116.84) (layer "F.SilkS")
+    (effects (font (size 1 1) (thickness 0.15)) (justify right))
+  )
   (gr_text "5V" (at 124.46 81.28) (layer "F.SilkS")
