File: PCB/relay/XRTL_PCB.kicad_pcb (KiCad board)
At the start: 2 copper layers, 63.5 x 86.4 mm, 28 parts, among them J10 servo1, J11 servo2, J12 infoLED, J13 USBC_5V_3A_input, J2 stepper1, J3 stepper2, J4 ESP32 right, J5 ESP32 left, K1 TIANBO-HJR-4102-L, K2 TIANBO-HJR-4102-L, U1 TBD62003, U2 TBD62003

Commit message: PCB updates
Other:
- board text added: "XRTL v1.1 Jari Domke 20/04/2023"
- board text removed: "XRTL v1.1 Jari Domke 25/01/2023"
Changed lines of the file:
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@@
       (layerselection 0x00010fc_ffffffff)
       (disableapertmacros false)
-      (usegerberextensions false)
-      (usegerberattributes true)
-      (usegerberadvancedattributes true)
-      (creategerberjobfile true)
+      (usegerberextensions true)
+      (usegerberattributes false)
+      (usegerberadvancedattributes false)
+      (creategerberjobfile false)
       (svguseinch false)
       (svgprecision 6)
@@
       (plotinvisibletext false)
       (sketchpadsonfab false)
-      (subtractmaskfromsilk false)
+      (subtractmaskfromsilk true)
       (outputformat 1)
       (mirror false)
@@
     (effects (font (size 1 1) (thickness 0.15)))
   )
-  (gr_text "XRTL v1.1\nJari Domke\n25/01/2023" (at 86.36 129.54) (layer "B.SilkS")
+  (gr_text "XRTL v1.1\nJari Domke\n20/04/2023" (at 86.36 129.54) (layer "B.SilkS")
     (effects (font (size 1 1) (thickness 0.15)) (justify left mirror))
   )
@@
     (effects (font (size 1 1) (thickness 0.15)))
   )
+  (gr_text "div" (at 124.46 116.84) (layer "F.SilkS")
+    (effects (font (size 1 1) (thickness 0.15)) (justify right))
+  )
   (gr_text "input" (at 124.46 114.3) (layer "F.SilkS")
